File: Insequor/PCB/KiCad/insequor58tray.kicad_pcb (KiCad board)
At the start: 2 copper layers, 173 x 143.5 mm, 103 parts, among them J1 Jumper, J2 Jumper

Commit message: Add files via upload
Connections:
- D1 pad 1: outerpinkie_bottom -> P21
- D10 pad 1: ring_middle -> P19
- D11 pad 1: ring_home -> P19
- D12 pad 1: ring_top -> P19
- D13 pad 1: middle_bottom -> P18
- D14 pad 1: middle_middle -> P18
- D15 pad 1: middle_home -> P18
- D16 pad 1: middle_top -> P18
- D17 pad 1: index_bottom -> P15
- D18 pad 1: index_middle -> P15
- D19 pad 1: index_home -> P15
- D2 pad 1: outerpinkie_middle -> P21
- D20 pad 1: index_top -> P15
- D21 pad 1: far_bottom -> P14
- D22 pad 1: far_middle -> P14
- D23 pad 1: far_home -> P14
- D24 pad 1: far_top -> P14
- D25 pad 1: first_bottom -> P21
- D26 pad 1: second_bottom -> P20
- D27 pad 1: third_bottom -> P19
- D28 pad 1: addon_bottom -> P18
- D29 pad 1: fourth_bottom -> P15
- D3 pad 1: outerpinkie_home -> P21
- D30 pad 1: fifth_bottom -> P14
- D4 pad 1: outerpinkie_top -> P21
- D5 pad 1: pinkie_bottom -> P20
- D6 pad 1: pinkie_middle -> P20
- D7 pad 1: pinkie_home -> P20
- D8 pad 1: pinkie_top -> P20
- D9 pad 1: ring_bottom -> P19
