File: Insequor/PCB/KiCad/insequor58≈Moon60.kicad_sch (KiCad schematic)
At the start: 74 parts, among them J3 OLED, SW1 SW_PUSH, SW10 SW_PUSH, SW11 SW_PUSH, SW12 SW_PUSH, SW13 SW_PUSH, SW14 SW_PUSH, SW15 SW_PUSH, SW16 SW_PUSH, SW17 SW_PUSH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

Commit message: KiCad update
Other:
- title: (none) -> Insequor58 ≈ Moon60
Changed lines of the file:
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@@
 (kicad_sch (version 20211123) (generator eeschema)
   (paper "A4")
+  (title_block
+    (title "Insequor58 ≈ Moon60")
+  )
   (junction (at 219.71 121.92) (diameter 0) (color 0 0 0 0)
   )
