File: Moon60/PCB/KiCad/insequor58≈Moon60.kicad_pcb (KiCad board)
At the start: 2 copper layers, 173 x 143.5 mm, 111 parts, among them J3 OLED

Commit message: KiCad files update
Parts:
- ? (x2): footprint (none) -> moon60Footprints:
- B1: footprint E73:SW_TACT_ALPS_SKQGABE010 -> moon60Footprints:SW_TACT_ALPS_SKQGABE010
- D1, D10, D11, D12, D13, D14, D15, D16, D17, D18, D19, D2, D20, D21, D22, D23, D24, D25, D26, D27, D28, D29, D3, D30, D4, D5, D6, D7, D8, D9: footprint ComboDiode -> moon60Footprints:ComboDiode
- G*** (x2): footprint Graphic:moonBIG -> moon60Footprints:moonBIG
- G*** (x2): footprint Graphic:moonMin -> moon60Footprints:moonMin
- J3: footprint Insequor58:OLED_4Pin -> moon60Footprints:OLED_4Pin
- JP1, JP2, JP3, JP4, JP5, JP6, JP7, JP8: footprint Insequor58:Jumper -> moon60Footprints:Jumper
- MCU1, MCU2: footprint ProMicro -> moon60Footprints:ProMicro
- R1 (x2): footprint Insequor58:RESISTOR_mini -> moon60Footprints:RESISTOR_mini
- REF**: footprint TRRS-PJ-320A-dual -> moon60Footprints:TRRS-PJ-320A-dual
- S1, S11, S13, S15, S17, S19, S21, S23, S25, S27, S29, S3, S31, S33, S35, S37, S39, S41, S43, S45, S47, S49, S5, S51, S53, S55, S57, S59, S7, S9: footprint PG1350 -> moon60Footprints:PG1350
- S10, S12, S14, S16, S18, S2, S20, S22, S24, S26, S28, S30, S32, S34, S36, S38, S4, S40, S42, S44, S46, S48, S50, S52, S54, S56, S58, S6, S60, S8: footprint MX -> moon60Footprints:MX
