File: Moon60/PCB/KiCad/insequor58≈Moon60.kicad_sch (KiCad schematic)
At the start: 74 parts, among them J3 OLED, SW1 SW_PUSH, SW10 SW_PUSH, SW11 SW_PUSH, SW12 SW_PUSH, SW13 SW_PUSH, SW14 SW_PUSH, SW15 SW_PUSH, SW16 SW_PUSH, SW17 SW_PUSH, SW18 SW_PUSH, SW19 SW_PUSH, SW2 SW_PUSH, SW20 SW_PUSH, SW21 SW_PUSH, SW22 SW_PUSH, SW23 SW_PUSH, SW24 SW_PUSH, SW25 SW_PUSH, SW26 SW_PUSH, SW27 SW_PUSH, SW28 SW_PUSH, SW29 SW_PUSH, SW3 SW_PUSH, SW30 SW_PUSH, SW4 SW_PUSH, SW5 SW_PUSH, SW6 SW_PUSH, SW7 SW_PUSH, SW8 SW_PUSH, SW9 SW_PUSH

Commit message: KiCad files update
Changed lines of the file:
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@@
   (junction (at 223.52 97.79) (diameter 0) (color 0 0 0 0)
   )
-  (junction (at 157.48 105.41) (diameter 0) (color 0 0 0 0)
-  )
   (junction (at 200.66 88.9) (diameter 0) (color 0 0 0 0)
   )
@@
     (stroke (width 0) (type default) (color 0 0 0 0))
   )
-  (wire (pts (xy 157.48 105.41) (xy 157.48 109.22))
-    (stroke (width 0) (type default) (color 0 0 0 0))
-  )
   (wire (pts (xy 238.76 72.39) (xy 257.81 72.39))
     (stroke (width 0) (type default) (color 0 0 0 0))
@@
     (stroke (width 0) (type default) (color 0 0 0 0))
   )
-  (wire (pts (xy 157.48 105.41) (xy 162.56 105.41))
-    (stroke (width 0) (type default) (color 0 0 0 0))
-  )
   (wire (pts (xy 111.76 59.69) (xy 120.65 59.69))
     (stroke (width 0) (type default) (color 0 0 0 0))
@@
     (stroke (width 0) (type default) (color 0 0 0 0))
   )
-  (wire (pts (xy 138.43 105.41) (xy 157.48 105.41))
-    (stroke (width 0) (type default) (color 0 0 0 0))
-  )
+  (wire (pts (xy 138.43 105.41) (xy 162.56 105.41))
+    (stroke (width 0) (type default) (color 0 0 0 0))
+  )
