File: 1.0/Moon60/PCB/KiCad/moon60NOi2c/insequor58≈Moon60NOi2c.kicad_pcb (KiCad board)
At the start: 2 copper layers, 173 x 143.5 mm, 110 parts, among them J2 4PIN, J3 OLED

Commit message: Moon60Symbols.kicad_sym
Parts:
- removed ? (x2): , moon60Footprints:
- added REF**: MountingHole_2.2mm_M2_ISO7380_Pad, MountingHole:MountingHole_2.2mm_M2_ISO7380_Pad, F.Cu at (264.2, 134.6)
- added REF**: MountingHole_2.2mm_M2_ISO7380_Pad, MountingHole:MountingHole_2.2mm_M2_ISO7380_Pad, F.Cu at (241.3, 134.6)
- B1 (x2): footprint moon60Footprints:SW_TACT_ALPS_SKQGABE010 -> Moon60footprints:SW_TACT_ALPS_SKQGABE010
- D1, D10, D11, D12, D13, D14, D15, D16, D17, D18, D19, D2, D20, D21, D22, D23, D24, D25, D26, D27, D28, D29, D3, D30, D4, D5, D6, D7, D8, D9: footprint moon60Footprints:ComboDiode -> Moon60footprints:ComboDiode
- G*** (x2): footprint moon60Footprints:moonBIG -> Moon60footprints:moonBIG
- G*** (x2): footprint moon60Footprints:moonMin -> Moon60footprints:moonMin
- J2: footprint Lily58-footprint:MJ-4PP-9 -> Moon60footprints:MJ-4PP-9
- J3: footprint moon60Footprints:OLED_4Pin -> Moon60footprints:OLED_4Pin
- JP1, JP2, JP3, JP4, JP5, JP6, JP7, JP8: footprint moon60Footprints:Jumper -> Moon60footprints:Jumper
- MCU1, MCU2: footprint moon60Footprints:ProMicro -> Moon60footprints:ProMicro
- S1, S11, S13, S15, S17, S19, S21, S23, S25, S27, S29, S3, S31, S33, S35, S37, S39, S41, S43, S45, S47, S49, S5, S51, S53, S55, S57, S59, S7, S9: footprint moon60Footprints:PG1350 -> Moon60footprints:PG1350
- S10, S12, S14, S16, S18, S2, S20, S22, S24, S26, S28, S30, S32, S34, S36, S38, S4, S40, S42, S44, S46, S48, S50, S52, S54, S56, S58, S6, S60, S8: footprint moon60Footprints:MX -> Moon60footprints:MX

Commit message: 1.0 PCB quick fix
Routing:
- net P6: track 486.7 -> 455.6 mm, vias 12 -> 7
- net P4: track 450.6 -> 420.6 mm, vias 12 -> 7
- net P5: track 467.7 -> 438.1 mm, vias 12 -> 7
- net P7: track 498.5 -> 470.9 mm, vias 12 -> 7
- net P8: track 483.9 -> 478.3 mm, vias 11 -> 8

Commit message: PCB manufacturing
Routing:
- net P8: track 478.3 -> 556.0 mm
- net P18: track 340.9 -> 396.3 mm, vias 7 -> 9
