File: 1.0/Moon60/PCB/KiCad/moon60NOi2c/insequor58≈Moon60Noi2c.kicad_sch (KiCad schematic)
At the start: 74 parts, among them J3 OLED, SW1 SW_PUSH, SW10 SW_PUSH, SW11 SW_PUSH, SW12 SW_PUSH, SW13 SW_PUSH, SW14 SW_PUSH, SW15 SW_PUSH, SW16 SW_PUSH, SW17 SW_PUSH, SW18 SW_PUSH, SW19 SW_PUSH, SW2 SW_PUSH, SW20 SW_PUSH, SW21 SW_PUSH, SW22 SW_PUSH, SW23 SW_PUSH, SW24 SW_PUSH, SW25 SW_PUSH, SW26 SW_PUSH, SW27 SW_PUSH, SW28 SW_PUSH, SW29 SW_PUSH, SW3 SW_PUSH, SW30 SW_PUSH, SW4 SW_PUSH, SW5 SW_PUSH, SW6 SW_PUSH, SW7 SW_PUSH, SW8 SW_PUSH, SW9 SW_PUSH

Commit message: Moon60Symbols.kicad_sym
Parts:
- removed J3: OLED, symbol kbd:OLED
- removed MCU1: ProMicro, symbol kbd:ProMicro
- removed R1, R2: R_Small, symbol Device:R_Small
- removed SW1, SW10, SW11, SW12, SW13, SW14, SW15, SW16, SW17, SW18, SW19, SW2, SW20, SW21, SW22, SW23, SW24, SW25, SW26, SW27, SW28, SW29, SW3, SW30, SW4, SW5, SW6, SW7, SW8, SW9: SW_PUSH, symbol kbd:SW_PUSH
- removed TRRS-PJ-320A-dual: MJ-4PP-9, symbol kbd:MJ-4PP-9
- added H1, H2: MountingHole_Pad, symbol Mechanical:MountingHole_Pad
- added J2: MJ-4PP-9, Moon60footprints:MJ-4PP-9, symbol Moon60Symbols:MJ-4PP-9
- added J3: OLED, Moon60footprints:OLED_4Pin, symbol Moon60Symbols:OLED
- added MCU1: ProMicro, Moon60footprints:ProMicro, symbol Moon60Symbols:ProMicro
- added SW1, SW10, SW11, SW12, SW13, SW14, SW15, SW16, SW17, SW18, SW19, SW2, SW20, SW21, SW22, SW23, SW24, SW25, SW26, SW27, SW28, SW29, SW3, SW30, SW4, SW5, SW6, SW7, SW8, SW9: SW_PUSH, symbol Moon60Symbols:SW_PUSH
- renumbered D15 to D10, D9 to D11, D3 to D12, D22 to D13, D16 to D14, D10 to D15, D4 to D16, D23 to D17, D17 to D18, D11 to D19, D5 to D20, D24 to D21, D18 to D22, D12 to D23, D6 to D24, D1 to D25, D21 to D9
Connections:
- net GND: now also J2.2, MCU1.15 (GND), MCU1.16 (GND), MCU1.2 (GND)
- net RESET: now also MCU1.3 (RST)
- net VCC: now also J2.1, MCU1.4 (VCC)
- net col1: now also MCU1.5 (F4/A3), SW1.1, SW2.1, SW25.1, SW3.1, SW4.1
- net col2: now also MCU1.6 (F5/A2), SW26.1, SW5.1, SW6.1, SW7.1, SW8.1
- net col3: now also MCU1.7 (F6/A1), SW10.1, SW11.1, SW12.1, SW27.1, SW9.1
- net col4: now also MCU1.8 (F7/A0), SW13.1, SW14.1, SW15.1, SW16.1, SW28.1
- net col5: now also MCU1.9 (B1/15), SW17.1, SW18.1, SW19.1, SW20.1, SW29.1
- net col6: now also MCU1.10 (B3/14), SW21.1, SW22.1, SW23.1, SW24.1, SW30.1
- net row1: now also MCU1.19 (4/D4)
- net row2: now also MCU1.20 (5/C6)
- net row3: now also MCU1.21 (6/D7)
- net row4: now also MCU1.22 (7/E6)
- net row5: now also MCU1.23 (8/B4)
- net at D24.1 (A): now also SW24.2
- net at D28.1 (A): now also SW28.2
- net at D1.1 (A): now also SW1.2
- net at D13.1 (A): now also SW13.2
- net at JP4.2 (B), JP5.2 (B): now also J3.1 (SDA)
- net at D25.1 (A): now also SW25.2
- net at D15.1 (A): now also SW15.2
- net at D10.1 (A): now also SW10.2
- net at D18.1 (A): now also SW18.2
- net at D29.1 (A): now also SW29.2
- net at JP3.2 (B), JP6.2 (B): now also J3.2 (SCL)
- net at D27.1 (A): now also SW27.2
- net at D4.1 (A): now also SW4.2
- net at D11.1 (A): now also SW11.2
- net at D2.1 (A): now also SW2.2
- net at D23.1 (A): now also SW23.2
- net at D8.1 (A): now also SW8.2
- net at D19.1 (A): now also SW19.2
- net at JP1.2 (B), JP8.2 (B): now also J3.4 (GND)
- net at D17.1 (A): now also SW17.2
- net at D21.1 (A): now also SW21.2
- net at D12.1 (A): now also SW12.2
- net at D9.1 (A): now also SW9.2
- net at D20.1 (A): now also SW20.2
- net at JP2.2 (B), JP7.2 (B): now also J3.3 (VCC)
- net at D22.1 (A): now also SW22.2
- net at D30.1 (A): now also SW30.2
- net at D3.1 (A): now also SW3.2
- net at D26.1 (A): now also SW26.2
- net at D14.1 (A): now also SW14.2
- net at D16.1 (A): now also SW16.2
- net at D7.1 (A): now also SW7.2
- net at D6.1 (A): now also SW6.2
- net at D5.1 (A): now also SW5.2
- new net DATA: J2.3, MCU1.14 (RX1/D2)
- no-connect marks 0 -> 1
Other:
- moved on the sheet: JP1, JP2, JP3, JP4, JP5, JP6, JP7, JP8

Commit message: kicad layers scan + minor changes to keymap
Other:
- company: (none) -> Wykonał: Przemysław Paciorek
Changed lines of the file:
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@@
   (title_block
     (title "Insequor58 ≈ Moon60")
+    (date "2022-11-02")
+    (company "Wykonał: Przemysław Paciorek")
   )
   (junction (at 219.71 121.92) (diameter 0) (color 0 0 0 0)
